Commit message: Add files via upload

File: crazyflie_description/urdf/crazy_fly.urdf (robot description, URDF)
Before this commit: robot crazyflie, 5 links, 4 joints
Links:
- added link imu_link, mass 0.01
- link base_link: geometry collision box size=0.095 0.095 0.02; visual box size=0.095 0.095 0.025
- link propeller_ccw_1: geometry collision cylinder length=0.004 radius=0.023; visual mesh filename=package://crazyflie_description/meshes/newwing_ccw.stl scale=0.001 0.001 0.001
- link propeller_ccw_3: geometry collision cylinder length=0.004 radius=0.023; visual mesh filename=package://crazyflie_description/meshes/newwing_ccw.stl scale=0.001 0.001 0.001
- link propeller_cw_2: geometry collision cylinder length=0.004 radius=0.023; visual mesh filename=package://crazyflie_description/meshes/newwing_cw.stl scale=0.001 0.001 0.001
- link propeller_cw_4: geometry collision cylinder length=0.004 radius=0.023; visual mesh filename=package://crazyflie_description/meshes/newwing_cw.stl scale=0.001 0.001 0.001
Joints:
- added joint imu_joint: type fixed, parent base_link, child imu_link, origin xyz=0 0 0
- joint joint_propeller_ccw_1: origin xyz=0.0316 0.0316 -0.0113 rpy=0 0 0 -> xyz=0.0316 0.0316 0.0113 rpy=0 0 0
- joint joint_propeller_ccw_3: origin xyz=-0.0316 -0.0316 -0.0113 rpy=0 0 0 -> xyz=-0.0316 -0.0316 0.0113 rpy=0 0 0
- joint joint_propeller_cw_2: axis 0 0 -1 -> 0 0 1; origin xyz=0.0316 -0.0316 -0.0113 rpy=0 0 0 -> xyz=0.0316 -0.0316 0.0113 rpy=0 0 0
- joint joint_propeller_cw_4: origin xyz=-0.0316 0.0316 -0.0113 rpy=0 0 0 -> xyz=-0.0316 0.0316 0.0113 rpy=0 0 0
